File: kicad/bats_less.kicad_pcb (KiCad board)
At the start: 2 copper layers, 26 parts, among them P1 SERVO, SW5 RESET, SW6 UP, SW7 LEFT, SW8 DOWN, SW9 RIGHT, U1 BUZZER

Commit message: Engadida unha "KiCAD cheat sheet", una chuleta para KiCAD, non rematada
Engadida unha segunda versión da placa intentando deixar todo nunha
cara.
Parts:
- moved R6 2.62 mm to (147.3, 128.9)
- moved R7 2.62 mm to (147.3, 123.8)
- moved SW5 2.54 mm to (132.1, 132.7)
Routing:
- net Net-(SHIELD1-PadRST): track 33.1 -> 39.8 mm
- net Net-(R6-Pad2): track 34.8 -> 33.1 mm
- net Net-(P1-Pad1): track 142.4 -> 141.7 mm
