File: kicad/bats.sch (KiCad schematic (older format))
At the start: 24 parts, among them P1 SERVO, SW1 RESET, SW2 SHOT, SW4 LEFT, SW6 RIGHT, U1 BUZZER

Commit message: Primeira versión completa con tres botóns. Os ficheiros gerber non son válidos. - Hai que revisar a conexión do servo - Hai que alinear ben os tres botóns
Parts:
- added LED5, LED6: LED, FT:LED-5MM, symbol LED
- added R10, R12: 220, extra:Resistor_Horizontal_SmallHole_RM10mm, symbol R
Connections:
- net ARD3: now also LED6.A; no longer R9.1, SW2.2
- net ARD4: now also LED5.A; no longer R11.1, SW4.2
- net GND: now also R10.2, R12.2
- net AD3: now reaches SHIELD1.AD3
- net AD3: now also R11.1, SW4.2
- net AD4: now reaches SHIELD1.AD4
- net AD4: now also R9.1, SW2.2
- net AD5: now reaches SHIELD1.AD5
- net AD5: now also R13.1, SW6.2
- removed net ARD2: R13.1, SHIELD1.2, SW6.2
- new net: LED5.K, R10.1
- new net: LED6.K, R12.1
- no-connect marks 19 -> 17
Other:
- moved on the sheet: LED2, LED3, R4, R5
Changed lines of the file:
@@
 L LED LED3
 U 1 1 55898085
-P 8150 1550
-F 0 "LED3" H 8150 1650 50  0000 C CNN
-F 1 "Green LED" H 8150 1450 50  0000 C CNN
-F 2 "FT:LED-5MM" H 8150 1550 60  0001 C CNN
-F 3 "" H 8150 1550 60  0000 C CNN
-	1    8150 1550
+P 8150 1400
+F 0 "LED3" H 8150 1500 50  0000 C CNN
+F 1 "Green LED" H 8150 1300 50  0000 C CNN
+F 2 "FT:LED-5MM" H 8150 1400 60  0001 C CNN
+F 3 "" H 8150 1400 60  0000 C CNN
+	1    8150 1400
 	1    0    0    -1
 $EndComp
@@
 L R R5
 U 1 1 55898121
-P 8700 1550
-F 0 "R5" V 8780 1550 50  0000 C CNN
-F 1 "220" V 8700 1550 50  0000 C CNN
-F 2 "extra:Resistor_Horizontal_SmallHole_RM10mm" H 8700 1550 60  0001 C CNN
-F 3 "" H 8700 1550 60  0000 C CNN
-	1    8700 1550
+P 8700 1400
+F 0 "R5" V 8780 1400 50  0000 C CNN
+F 1 "220" V 8700 1400 50  0000 C CNN
+F 2 "extra:Resistor_Horizontal_SmallHole_RM10mm" H 8700 1400 60  0001 C CNN
+F 3 "" H 8700 1400 60  0000 C CNN
+	1    8700 1400
 	0    -1   -1   0
 $EndComp
@@
 L LED LED2
 U 1 1 55898212
-P 8150 1150
-F 0 "LED2" H 8150 1250 50  0000 C CNN
-F 1 "Yellow LED" H 8150 1050 50  0000 C CNN
-F 2 "FT:LED-5MM" H 8150 1150 60  0001 C CNN
-F 3 "" H 8150 1150 60  0000 C CNN
-	1    8150 1150
+P 8150 1075
+F 0 "LED2" H 8150 1175 50  0000 C CNN
+F 1 "Yellow LED" H 8150 975 50  0000 C CNN
+F 2 "FT:LED-5MM" H 8150 1075 60  0001 C CNN
+F 3 "" H 8150 1075 60  0000 C CNN
+	1    8150 1075
 	1    0    0    -1
 $EndComp
@@
 L R R4
 U 1 1 55898218
-P 8700 1150
-F 0 "R4" V 8780 1150 50  0000 C CNN
-F 1 "220" V 8700 1150 50  0000 C CNN
-F 2 "extra:Resistor_Horizontal_SmallHole_RM10mm" H 8700 1150 60  0001 C CNN
-F 3 "" H 8700 1150 60  0000 C CNN
-	1    8700 1150
+P 8700 1075
+F 0 "R4" V 8780 1075 50  0000 C CNN
+F 1 "220" V 8700 1075 50  0000 C CNN
+F 2 "extra:Resistor_Horizontal_SmallHole_RM10mm" H 8700 1075 60  0001 C CNN
+F 3 "" H 8700 1075 60  0000 C CNN
+	1    8700 1075
 	0    -1   -1   0
 $EndComp
@@
 L GND #PWR08
 U 1 1 558C0B72
-P 9400 1250
-F 0 "#PWR08" H 9400 1000 50  0001 C CNN
-F 1 "GND" H 9400 1100 50  0000 C CNN
-F 2 "" H 9400 1250 60  0000 C CNN
-F 3 "" H 9400 1250 60  0000 C CNN
-	1    9400 1250
+P 9400 1175
+F 0 "#PWR08" H 9400 925 50  0001 C CNN
+F 1 "GND" H 9400 1025 50  0000 C CNN
+F 2 "" H 9400 1175 60  0000 C CNN
+F 3 "" H 9400 1175 60  0000 C CNN
+	1    9400 1175
 	1    0    0    -1
 $EndComp
@@
 GND3
 Wire Wire Line
-	8450 1550 8350 1550
-Wire Wire Line
-	8450 1150 8350 1150
+	8450 1400 8350 1400
+Wire Wire Line
+	8450 1075 8350 1075
 Wire Wire Line
 	8450 750  8350 750
@@
 	1000 2000 1000 2100
 Wire Wire Line
-	9100 1550 8950 1550
-Wire Wire Line
-	9100 750  9100 1550
+	9100 1400 8950 1400
+Wire Wire Line
+	9100 750  9100 2050
 Wire Wire Line
 	9100 750  8950 750
 Wire Wire Line
-	8950 1150 9400 1150
-Connection ~ 9100 1150
+	8950 1075 9400 1075
+Connection ~ 9100 1075
 Wire Wire Line
 	1000 2600 1000 2750
@@
 	10550 2850 10550 3000
 Wire Wire Line
-	9400 1150 9400 1250
+	9400 1075 9400 1175
 Wire Wire Line
 	7400 5550 7600 5550
@@
 	0    1    1    0
 $EndComp
-NoConn ~ 4850 4650
 $Comp
 L ARDUINO_SHIELD SHIELD1
@@
 	7950 750  7550 750
 Wire Wire Line
-	7950 1150 7550 1150
-Wire Wire Line
-	7950 1550 7550 1550
+	7950 1075 7550 1075
+Wire Wire Line
+	7950 1400 7550 1400
 Text Label 6750 3650 0    60   ~ 0
 ARD11
@@
 Text Label 8550 2700 2    60   ~ 0
 ARD11
-Text Label 7550 1150 2    60   ~ 0
+Text Label 7550 1075 2    60   ~ 0
 ARD7
 Text Label 7550 750  2    60   ~ 0
 ARD8
-Text Label 7550 1550 2    60   ~ 0
+Text Label 7550 1400 2    60   ~ 0
 ARD6
 Text Label 6750 4250 0    60   ~ 0
@@
 Wire Wire Line
 	9300 5450 9300 5600
-Text Label 6750 4650 0    60   ~ 0
-ARD2
 Text Label 6750 4550 0    60   ~ 0
 ARD3
@@
 	10500 4650 8950 4650
 Text Label 8950 4650 2    60   ~ 0
-ARD2
+AD5
 Connection ~ 9900 4750
 Wire Wire Line
 	9900 4750 8450 4750
 Text Label 8450 4750 2    60   ~ 0
-ARD4
+AD3
 Connection ~ 9300 4850
 Wire Wire Line
 	9300 4850 7950 4850
 Text Label 7950 4850 2    60   ~ 0
-ARD3
+AD4
 Text Label 4850 3850 2    60   ~ 0
 VCC
@@
 Text Label 4850 4550 2    60   ~ 0
 AD2
-NoConn ~ 4850 4750
-NoConn ~ 4850 4850
 Text Label 6750 4350 0    60   ~ 0
 ARD5
+Text Label 4850 4650 2    60   ~ 0
+AD3
+Text Label 4850 4750 2    60   ~ 0
+AD4
+Text Label 4850 4850 2    60   ~ 0
+AD5
+$Comp
+L LED LED5
+U 1 1 57448A7A
+P 8150 1725
+F 0 "LED5" H 8150 1825 50  0000 C CNN
+F 1 "LED" H 8150 1625 50  0000 C CNN
+F 2 "FT:LED-5MM" H 8150 1725 60  0001 C CNN
+F 3 "" H 8150 1725 60  0000 C CNN
+	1    8150 1725
+	1    0    0    -1
+$EndComp
+$Comp
+L R R10
+U 1 1 57448A80
+P 8700 1725
+F 0 "R10" V 8780 1725 50  0000 C CNN
+F 1 "220" V 8700 1725 50  0000 C CNN
+F 2 "extra:Resistor_Horizontal_SmallHole_RM10mm" H 8700 1725 60  0001 C CNN
+F 3 "" H 8700 1725 60  0000 C CNN
+	1    8700 1725
+	0    -1   -1   0
+$EndComp
+Wire Wire Line
+	8450 1725 8350 1725
+Wire Wire Line
+	9100 1725 8950 1725
+Wire Wire Line
+	7950 1725 7550 1725
+Text Label 7550 1725 2    60   ~ 0
+ARD4
+$Comp
+L LED LED6
+U 1 1 57448B75
+P 8150 2050
+F 0 "LED6" H 8150 2150 50  0000 C CNN
+F 1 "LED" H 8150 1950 50  0000 C CNN
+F 2 "FT:LED-5MM" H 8150 2050 60  0001 C CNN
+F 3 "" H 8150 2050 60  0000 C CNN
+	1    8150 2050
+	1    0    0    -1
+$EndComp
+$Comp
+L R R12
+U 1 1 57448B7B
+P 8700 2050
+F 0 "R12" V 8780 2050 50  0000 C CNN
+F 1 "220" V 8700 2050 50  0000 C CNN
+F 2 "extra:Resistor_Horizontal_SmallHole_RM10mm" H 8700 2050 60  0001 C CNN
+F 3 "" H 8700 2050 60  0000 C CNN
+	1    8700 2050
+	0    -1   -1   0
+$EndComp
+Wire Wire Line
+	8450 2050 8350 2050
+Wire Wire Line
+	9100 2050 8950 2050
+Wire Wire Line
+	7950 2050 7550 2050
+Text Label 7550 2050 2    60   ~ 0
+ARD3
+Connection ~ 9100 1400
+Connection ~ 9100 1725
+NoConn ~ 6750 4650
 $EndSCHEMATC

Commit message: Engadida a biblioteca KiCAD de BricoLabs coma submodule
Parts:
- VR1, VR2: footprint FT:POT_RV09_VERT -> bl_kicad:POT_RV09_VERT_easySoldering
Changed lines of the file:
@@
 LIBS:contrib
 LIBS:valves
+LIBS:bl_kicad
 LIBS:bats-cache
 EELAYER 25 0
@@
 F 0 "VR1" H 2200 4350 50  0000 C CNN
 F 1 "POT" H 2200 4450 50  0000 C CNN
-F 2 "FT:POT_RV09_VERT" H 2200 4450 60  0001 C CNN
+F 2 "bl_kicad:POT_RV09_VERT_easySoldering" H 2200 4450 60  0001 C CNN
 F 3 "" H 2200 4450 60  0000 C CNN
 	1    2200 4450
@@
 F 0 "VR2" H 2650 4650 50  0000 C CNN
 F 1 "POT" H 2650 4750 50  0000 C CNN
-F 2 "FT:POT_RV09_VERT" H 2650 4750 60  0001 C CNN
+F 2 "bl_kicad:POT_RV09_VERT_easySoldering" H 2650 4750 60  0001 C CNN
 F 3 "" H 2650 4750 60  0000 C CNN
 	1    2650 4750

Commit message: Engadidas as novas pisadas "easy soldering" dende a biblioteca KiCAD de BricoLabs Actualizados os submódulos
Parts:
- LED1, LED2, LED3, LED5, LED6: footprint FT:LED-5MM -> bl_kicad:LED-5MM_easy_soldering
Changed lines of the file:
@@
 F 0 "LED3" H 8150 1500 50  0000 C CNN
 F 1 "Green LED" H 8150 1300 50  0000 C CNN
-F 2 "FT:LED-5MM" H 8150 1400 60  0001 C CNN
+F 2 "bl_kicad:LED-5MM_easy_soldering" H 8150 1400 60  0001 C CNN
 F 3 "" H 8150 1400 60  0000 C CNN
 	1    8150 1400
@@
 F 0 "LED2" H 8150 1175 50  0000 C CNN
 F 1 "Yellow LED" H 8150 975 50  0000 C CNN
-F 2 "FT:LED-5MM" H 8150 1075 60  0001 C CNN
+F 2 "bl_kicad:LED-5MM_easy_soldering" H 8150 1075 60  0001 C CNN
 F 3 "" H 8150 1075 60  0000 C CNN
 	1    8150 1075
@@
 F 0 "LED1" H 8150 850 50  0000 C CNN
 F 1 "Red LED" H 8150 650 50  0000 C CNN
-F 2 "FT:LED-5MM" H 8150 750 60  0001 C CNN
+F 2 "bl_kicad:LED-5MM_easy_soldering" H 8150 750 60  0001 C CNN
 F 3 "" H 8150 750 60  0000 C CNN
 	1    8150 750
@@
 F 0 "LED5" H 8150 1825 50  0000 C CNN
 F 1 "LED" H 8150 1625 50  0000 C CNN
-F 2 "FT:LED-5MM" H 8150 1725 60  0001 C CNN
+F 2 "bl_kicad:LED-5MM_easy_soldering" H 8150 1725 60  0001 C CNN
 F 3 "" H 8150 1725 60  0000 C CNN
 	1    8150 1725
@@
 F 0 "LED6" H 8150 2150 50  0000 C CNN
 F 1 "LED" H 8150 1950 50  0000 C CNN
-F 2 "FT:LED-5MM" H 8150 2050 60  0001 C CNN
+F 2 "bl_kicad:LED-5MM_easy_soldering" H 8150 2050 60  0001 C CNN
 F 3 "" H 8150 2050 60  0000 C CNN
 	1    8150 2050

Commit message: Revisados adornos dos silks e números de versións
Parts:
- LED4: footprint FT:LED-RGB-8MM-COM-K-MINIMAL -> bl_kicad:LED-RGB-8MM-COM-K-MINIMAL_easy_soldering
Changed lines of the file:
@@
 Sheet 1 1
 Title "BATS: BricoLabs Arduino Training Shield"
-Date "2016-01-05"
-Rev "2.0"
+Date "2017-09-27"
+Rev "3.0"
 Comp "BricoLabs"
 Comment1 ""
@@
 F 0 "LED4" H 9550 2800 50  0000 C CNN
 F 1 "LED_RGB_COM_K" H 9750 2300 50  0000 C CNN
-F 2 "FT:LED-RGB-8MM-COM-K-MINIMAL" H 9700 2700 60  0001 C CNN
+F 2 "bl_kicad:LED-RGB-8MM-COM-K-MINIMAL_easy_soldering" H 9700 2700 60  0001 C CNN
 F 3 "" H 9700 2700 60  0000 C CNN
 	1    9700 2700
